File: Hardware/MicroSD_Sniffer.sch (EAGLE design)
At the start: 9 parts, among them U1 MICRO-SDCARD, U2 microSD Socket

Commit message: Official QC checklist items
Other:
- note added: "Tim Holmberg"
- note added: "V01"
- note removed: "V10"
Changed lines of the file:
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@@
 <plain>
 <text x="104.14" y="73.66" size="1.778" layer="97">PCB must be no thicker than 0.75mm</text>
-<text x="238.76" y="7.62" size="2.54" layer="94">V10</text>
+<text x="238.76" y="7.62" size="2.54" layer="94">V01</text>
 <text x="148.336" y="6.604" size="2.54" layer="94">Revised by: Patrick Alberts</text>
+<text x="165.608" y="11.43" size="2.54" layer="94">Tim Holmberg</text>
 </plain>
 <instances>
@@
 <attribute name="VALUE" x="227.076" y="84.074" size="1.778" layer="96" rot="R180"/>
 </instance>
-<instance part="LOGO1" gate="G$1" x="233.68" y="45.72"/>
-<instance part="LOGO2" gate="G$1" x="211.582" y="37.592"/>
-<instance part="LOGO3" gate="G$1" x="148.59" y="32.766"/>
+<instance part="LOGO1" gate="G$1" x="223.52" y="45.72"/>
+<instance part="LOGO2" gate="G$1" x="203.962" y="37.592"/>
+<instance part="LOGO3" gate="G$1" x="143.51" y="32.766"/>
 <instance part="U1" gate="G$1" x="38.1" y="93.98"/>
-<instance part="FID1" gate="G$1" x="246.38" y="33.02"/>
-<instance part="FID2" gate="G$1" x="241.3" y="33.02"/>
+<instance part="FID1" gate="G$1" x="241.3" y="38.1"/>
+<instance part="FID2" gate="G$1" x="246.38" y="38.1"/>
 <instance part="GND1" gate="1" x="139.7" y="96.52"/>
 <instance part="GND2" gate="1" x="71.12" y="96.52"/>
@@
 <pinref part="GND3" gate="1" pin="GND"/>
 <wire x1="187.96" y1="106.68" x2="187.96" y2="96.52" width="0.1524" layer="91"/>
-<wire x1="187.96" y1="96.52" x2="187.96" y2="91.44" width="0.1524" layer="91"/>
+<wire x1="187.96" y1="96.52" x2="187.96" y2="93.98" width="0.1524" layer="91"/>
+<wire x1="187.96" y1="93.98" x2="187.96" y2="91.44" width="0.1524" layer="91"/>
 <wire x1="187.96" y1="91.44" x2="187.96" y2="88.9" width="0.1524" layer="91"/>
 <wire x1="187.96" y1="88.9" x2="187.96" y2="83.82" width="0.1524" layer="91"/>
@@
 <wire x1="203.2" y1="88.9" x2="187.96" y2="88.9" width="0.1524" layer="91"/>
 <junction x="187.96" y="88.9"/>
+<wire x1="203.2" y1="93.98" x2="187.96" y2="93.98" width="0.1524" layer="91"/>
+<pinref part="U2" gate="G$1" pin="CD1"/>
+<junction x="187.96" y="93.98"/>
 </segment>
 <segment>
-<wire x1="203.2" y1="93.98" x2="187.96" y2="93.98" width="0.1524" layer="91"/>
-<pinref part="U2" gate="G$1" pin="CD1"/>
-</segment>
-<segment>

Commit message: changed fids to regular
Parts:
- FID1, FID2: value FIDUCIALUFIDUCIAL -> FIDUCIAL1X2; device SparkFun-Aesthetics:FIDUCIALUFIDUCIAL -> SparkFun-Aesthetics:FIDUCIAL1X2
Changed lines of the file:
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@@
 <?xml version="1.0" encoding="utf-8"?>
 <!DOCTYPE eagle SYSTEM "eagle.dtd">
-<eagle version="6.4">
+<eagle version="6.6.0">
 <drawing>
 <settings>
@@
 <part name="LOGO3" library="SparkFun-Aesthetics" deviceset="SFE_LOGO_NAME_FLAME" device=".1_INCH"/>
 <part name="U1" library="SparkFun-Boards" deviceset="MICRO-SDCARD" device=""/>
-<part name="FID1" library="SparkFun-Aesthetics" deviceset="FIDUCIAL" device="UFIDUCIAL"/>
-<part name="FID2" library="SparkFun-Aesthetics" deviceset="FIDUCIAL" device="UFIDUCIAL"/>
 <part name="GND1" library="SparkFun-Aesthetics" deviceset="GND" device=""/>
 <part name="GND2" library="SparkFun-Aesthetics" deviceset="GND" device=""/>
@@
 <part name="GND3" library="SparkFun-Aesthetics" deviceset="GND" device=""/>
 <part name="SUPPLY3" library="SparkFun-Aesthetics" deviceset="VCC" device=""/>
+<part name="FID1" library="SparkFun-Aesthetics" deviceset="FIDUCIAL" device="1X2"/>
+<part name="FID2" library="SparkFun-Aesthetics" deviceset="FIDUCIAL" device="1X2"/>
 </parts>
 <sheets>
@@
 <instance part="LOGO3" gate="G$1" x="143.51" y="32.766"/>
 <instance part="U1" gate="G$1" x="38.1" y="93.98"/>
-<instance part="FID1" gate="G$1" x="241.3" y="38.1"/>
-<instance part="FID2" gate="G$1" x="246.38" y="38.1"/>
 <instance part="GND1" gate="1" x="139.7" y="96.52"/>
 <instance part="GND2" gate="1" x="71.12" y="96.52"/>
@@
 <instance part="GND3" gate="1" x="187.96" y="81.28"/>
 <instance part="SUPPLY3" gate="G$1" x="187.96" y="121.92"/>
+<instance part="FID1" gate="G$1" x="241.3" y="38.1"/>
+<instance part="FID2" gate="G$1" x="246.38" y="38.1"/>
 </instances>
 <busses>
